File: kicad/fuzz-effect/fuzz-effect.kicad_pcb (KiCad board)
At the start: 2 copper layers, 79.5 x 45.5 mm, 16 parts, among them J1 NMJ4HHD2, J2 NMJ4HHD2, J3 Screw_Terminal_01x02, Q1 BC337

Commit message: Add single-transistor-voltage-amplifier-negative-feedback and update readme
Parts:
- C1, C3, C5: value C -> 100n
- C2, C4: value C -> 10n
- C6: value C -> 22u
- R1, R2: value R -> 100k
- R3: value R -> 470
- R4: value R -> 51k
Changed lines of the file:
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@@
 			)
 		)
-		(property "Value" "C"
+		(property "Value" "100n"
 			(at 1.25 2 0)
 			(layer "F.Fab")
@@
 			)
 		)
-		(property "Value" "R"
+		(property "Value" "51k"
 			(at 0.95 1.92 0)
 			(layer "F.Fab")
@@
 			)
 		)
-		(property "Value" "C"
+		(property "Value" "22u"
 			(at 1.25 2.3 90)
 			(layer "F.Fab")
@@
 			)
 		)
-		(property "Value" "C"
+		(property "Value" "100n"
 			(at 1.25 2.3 0)
 			(layer "F.Fab")
@@
 			)
 		)
-		(property "Value" "R"
+		(property "Value" "470"
 			(at 0.95 1.92 90)
 			(layer "F.Fab")
@@
 			)
 		)
-		(property "Value" "C"
+		(property "Value" "10n"
 			(at 1.25 2.3 90)
 			(layer "F.Fab")
@@
 			)
 		)
-		(property "Value" "C"
+		(property "Value" "10n"
 			(at 1.25 2.3 0)
 			(layer "F.Fab")
@@
 			)
 		)
-		(property "Value" "R"
+		(property "Value" "100k"
 			(at 0.95 1.92 0)
 			(layer "F.Fab")
@@
 			)
 		)
-		(property "Value" "R"
+		(property "Value" "100k"
 			(at 0.95 1.92 0)
 			(layer "F.Fab")
@@
 			)
 		)
-		(property "Value" "C"
+		(property "Value" "100n"
 			(at 1.25 2.3 90)
 			(layer "F.Fab")
